File: hardware/kicad/Circuit layout.kicad_sch (KiCad schematic)
At the start: 79 parts, among them U1 TPS7A2025PDQNR, U2 LM27761, U3 ADS1299IPAGR, U4 nRF52832-QFxx, Y1 32MHz

Commit message: Added footprints - Dillon
Added footprints, symbols and 3d models

Now need to update with new antenna
Parts:
- U1: footprint EEG chips:TPS7A2025PDQNR -> foots:TPS7A2025PDQNR
- U2: footprint EEG chips:LM27761DSGT -> foots:LM27761DSGT
- U3: footprint EEG chips:ADS1299IPAGR -> foots:ADS1299IPAGR
- U4: footprint EEG chips:nRF52832-QFAA-R -> foots:NRF52832-QFAA-R
Connections:
- net at C12.2, R8.1, U3.15 (IN1N): now also C10.1, C11.1, C9.1, R10.2, R11.2, R9.2, U3.11 (IN3N), U3.13 (IN2N), U3.9 (IN4N)
Other:
- moved on the sheet: AE1, C1, C2, C27, C28, C29, C30, C31, C32, C33, C34, C7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

Commit message: test points added
also, antenna added, component numbering done, all footprints there, need to populate BOM
Parts:
- removed AE1: Antenna_Chip, RF_Antenna:Johanson_2450AT18x100, symbol Device:Antenna_Chip
- removed C34: 1pF, Capacitor_SMD:C_0603_1608Metric_Pad1.08x0.95mm_HandSolder, symbol Device:C
- removed R6: 4.99K, Resistor_SMD:R_0402_1005Metric_Pad0.72x0.64mm_HandSolder, symbol Device:R
- removed TP11: SWDIO, symbol Connector:TestPoint
- removed TP12: SWDCLK, symbol Connector:TestPoint
- removed TP13: +2V5, symbol Connector:TestPoint
- added C10, C9: 4.7nF, Capacitor_SMD:C_0402_1005Metric_Pad0.74x0.62mm_HandSolder, symbol Device:C
- added C27: 0p3, Capacitor_SMD:C_0402_1005Metric, symbol Device:C
- added C28: 0p8, Capacitor_SMD:C_0402_1005Metric, symbol Device:C
- added FLT1: DLF162500LT-5028A1, foots:DLF162500LT-5028A1, symbol Bluephildemo_projlib:DLF162500LT-5028A1
- added FM1, FM2, FM3: Fiducial, Fiducial:Fiducial_1mm_Mask2mm, symbol Mechanical:Fiducial
- added H1, H2, H3, H4: MountingHole_Pad, MountingHole:MountingHole_2.2mm_M2_Pad_Via, symbol Mechanical:MountingHole_Pad
- added L4: AMCA31-2R450G-S1F-T3, foots:AMCA31-2R450G-S1F-T3, symbol AMCA31-2R450G-S1F-T3:AMCA31-2R450G-S1F-T3
- added R3: 4.99K, Resistor_SMD:R_0402_1005Metric_Pad0.72x0.64mm_HandSolder, symbol Device:R
- added TP1: PWR, TestPoint:TestPoint_THTPad_2.5x2.5mm_Drill1.2mm, symbol Connector:TestPoint
- added TP17: CS_ADS, TestPoint:TestPoint_THTPad_2.5x2.5mm_Drill1.2mm, symbol Connector:TestPoint
- added TP18: RESET_ADS, TestPoint:TestPoint_THTPad_2.5x2.5mm_Drill1.2mm, symbol Connector:TestPoint
- added TP19: MOSI_ADS, TestPoint:TestPoint_THTPad_2.5x2.5mm_Drill1.2mm, symbol Connector:TestPoint
- added TP20: P21, TestPoint:TestPoint_THTPad_2.5x2.5mm_Drill1.2mm, symbol Connector:TestPoint
- added TP21: SWDCLK, TestPoint:TestPoint_THTPad_2.5x2.5mm_Drill1.2mm, symbol Connector:TestPoint
- added TP22: SWDIO, TestPoint:TestPoint_THTPad_2.5x2.5mm_Drill1.2mm, symbol Connector:TestPoint
- added TP23: P0, TestPoint:TestPoint_THTPad_2.5x2.5mm_Drill1.2mm, symbol Connector:TestPoint
- added TP24: P1, TestPoint:TestPoint_THTPad_2.5x2.5mm_Drill1.2mm, symbol Connector:TestPoint
- added TP25: P2, TestPoint:TestPoint_THTPad_2.5x2.5mm_Drill1.2mm, symbol Connector:TestPoint
- added TP26: P3, TestPoint:TestPoint_THTPad_2.5x2.5mm_Drill1.2mm, symbol Connector:TestPoint
- added TP27: DRDY_NRF, TestPoint:TestPoint_THTPad_2.5x2.5mm_Drill1.2mm, symbol Connector:TestPoint
- added TP28: MISO_NRF, TestPoint:TestPoint_THTPad_2.5x2.5mm_Drill1.2mm, symbol Connector:TestPoint
- added TP29: P6, TestPoint:TestPoint_THTPad_2.5x2.5mm_Drill1.2mm, symbol Connector:TestPoint
- added TP3: 2.5V, TestPoint:TestPoint_THTPad_2.5x2.5mm_Drill1.2mm, symbol Connector:TestPoint
- added TP30: CS_NRF, TestPoint:TestPoint_THTPad_2.5x2.5mm_Drill1.2mm, symbol Connector:TestPoint
- added TP31: RESET_NRF, TestPoint:TestPoint_THTPad_2.5x2.5mm_Drill1.2mm, symbol Connector:TestPoint
- added TP32: MOSI_NRF, TestPoint:TestPoint_THTPad_2.5x2.5mm_Drill1.2mm, symbol Connector:TestPoint
- added TP33: P10, TestPoint:TestPoint_THTPad_2.5x2.5mm_Drill1.2mm, symbol Connector:TestPoint
- added TP34: SCLK_NRF, TestPoint:TestPoint_THTPad_2.5x2.5mm_Drill1.2mm, symbol Connector:TestPoint
- added TP35: P12, TestPoint:TestPoint_THTPad_2.5x2.5mm_Drill1.2mm, symbol Connector:TestPoint
- added TP36: P13, TestPoint:TestPoint_THTPad_2.5x2.5mm_Drill1.2mm, symbol Connector:TestPoint
- added TP37: P14, TestPoint:TestPoint_THTPad_2.5x2.5mm_Drill1.2mm, symbol Connector:TestPoint
- added TP38: P15, TestPoint:TestPoint_THTPad_2.5x2.5mm_Drill1.2mm, symbol Connector:TestPoint
- added TP39: P16, TestPoint:TestPoint_THTPad_2.5x2.5mm_Drill1.2mm, symbol Connector:TestPoint
- added TP40: P17, TestPoint:TestPoint_THTPad_2.5x2.5mm_Drill1.2mm, symbol Connector:TestPoint
- added TP41: P18, TestPoint:TestPoint_THTPad_2.5x2.5mm_Drill1.2mm, symbol Connector:TestPoint
- added TP42: P19, TestPoint:TestPoint_THTPad_2.5x2.5mm_Drill1.2mm, symbol Connector:TestPoint
- added TP43: P20, TestPoint:TestPoint_THTPad_2.5x2.5mm_Drill1.2mm, symbol Connector:TestPoint
- added TP44: P22, TestPoint:TestPoint_THTPad_2.5x2.5mm_Drill1.2mm, symbol Connector:TestPoint
- added TP45: P23, TestPoint:TestPoint_THTPad_2.5x2.5mm_Drill1.2mm, symbol Connector:TestPoint
- added TP46: P24, TestPoint:TestPoint_THTPad_2.5x2.5mm_Drill1.2mm, symbol Connector:TestPoint
- added TP47: P25, TestPoint:TestPoint_THTPad_2.5x2.5mm_Drill1.2mm, symbol Connector:TestPoint
- added TP48: P26, TestPoint:TestPoint_THTPad_2.5x2.5mm_Drill1.2mm, symbol Connector:TestPoint
- added TP49: P27, TestPoint:TestPoint_THTPad_2.5x2.5mm_Drill1.2mm, symbol Connector:TestPoint
- added TP5: EEG7, TestPoint:TestPoint_THTPad_2.5x2.5mm_Drill1.2mm, symbol Connector:TestPoint
- added TP50: P28, TestPoint:TestPoint_THTPad_2.5x2.5mm_Drill1.2mm, symbol Connector:TestPoint
- added TP51: P29, TestPoint:TestPoint_THTPad_2.5x2.5mm_Drill1.2mm, symbol Connector:TestPoint
- added TP52: P30, TestPoint:TestPoint_THTPad_2.5x2.5mm_Drill1.2mm, symbol Connector:TestPoint
- added TP53: P31, TestPoint:TestPoint_THTPad_2.5x2.5mm_Drill1.2mm, symbol Connector:TestPoint
- L3: value 3.9nH -> 2n7; footprint Inductor_SMD:L_0402_1005Metric_Pad0.77x0.64mm_HandSolder -> Inductor_SMD:L_0402_1005Metric; Distributor Link (none) -> https://www.mouser.co.uk/ProductDetail/Murata-Electronics/L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; Manufacturer (none) -> Murata; Manufacturer Part Number (none) -> LQG15HS2N7S02D
- TP10: renamed from TP7; footprint (none) -> TestPoint:TestPoint_THTPad_2.5x2.5mm_Drill1.2mm
- TP11: renamed from TP8; footprint (none) -> TestPoint:TestPoint_THTPad_2.5x2.5mm_Drill1.2mm
- TP12: renamed from TP9; footprint (none) -> TestPoint:TestPoint_THTPad_2.5x2.5mm_Drill1.2mm
- TP13: renamed from TP10; footprint (none) -> TestPoint:TestPoint_THTPad_2.5x2.5mm_Drill1.2mm
- TP14: value -2V5 -> DRDY_ADS; footprint (none) -> TestPoint:TestPoint_THTPad_2.5x2.5mm_Drill1.2mm
- TP15: value +BATT -> MISO_ADS; footprint (none) -> TestPoint:TestPoint_THTPad_2.5x2.5mm_Drill1.2mm
- TP16: value GND -> SCLK_ADS; footprint (none) -> TestPoint:TestPoint_THTPad_2.5x2.5mm_Drill1.2mm
- TP2: value EOGV_P -> 2.5V; footprint (none) -> TestPoint:TestPoint_THTPad_2.5x2.5mm_Drill1.2mm
- TP4: value EOGH_P -> EEG8; footprint (none) -> TestPoint:TestPoint_THTPad_2.5x2.5mm_Drill1.2mm
- TP6: renamed from TP1; value EOGV_N -> EEG6; footprint (none) -> TestPoint:TestPoint_THTPad_2.5x2.5mm_Drill1.2mm
- TP7: renamed from TP3; value EOGH_N -> EEG5; footprint (none) -> TestPoint:TestPoint_THTPad_2.5x2.5mm_Drill1.2mm
- TP8: renamed from TP5; footprint (none) -> TestPoint:TestPoint_THTPad_2.5x2.5mm_Drill1.2mm
- TP9: renamed from TP6; footprint (none) -> TestPoint:TestPoint_THTPad_2.5x2.5mm_Drill1.2mm
- renumbered C9 to C11, C10 to C12, C11 to C13, C12 to C14, C18 to C15, C19 to C16, C20 to C17, C21 to C18, C22 to C19, C27 to C20, C26 to C21, C25 to C22, C28 to C23, C29 to C24, C30 to C25, C31 to C26, C33 to C29, C4 to C3, C32 to C30, C13 to C31, C14 to C32, C15 to C34, C16 to C35, C17 to C36, C23 to C37, C24 to C38, C3 to C4, L2 to L1, L1 to L2, R2 to R1, R8 to R10, R7 to R11, R20 to R12, R19 to R13, R18 to R13, R16 to R14, R14 to R16, R13 to R17, R17 to R18, R12 to R19, R1 to R2, R3 to R5, R5 to R6, R11 to R7, R10 to R8
Connections:
- net +2V5: now also TP2.1; no longer U3.1 (IN8N), U3.2 (IN8P), U3.3 (IN7N), U3.4 (IN7P)
- net -2V5: now also TP3.1; no longer TP14.1
- net GND: now also C29.2, C30.2, Y1.4, C27.2, C28.2, FLT1.2 (GND), FLT1.4 (GND), H1.1, H2.1, H3.1, H4.1, L4.1 (FEED); no longer TP16.1
- net at C11.2, C12.2, C13.2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: now also C7.2, C8.2, C10.2, C9.2
- net at TP4.1: now also R3.1
- net at R5.2, U3.5 (IN6N): now also C9.1; no longer C7.1
- net at R6.2, U3.7 (IN5N): now also C10.1; no longer C8.1
- net at U3.8 (IN5P): no longer C8.2
- net at U4.12 (NFC2/P0.10): now also TP33.1
- net at U4.15 (P0.12): now also TP35.1
- net at U4.16 (P0.13): now also TP36.1
- net at U4.17 (P0.14): now also TP37.1
- net at U4.18 (P0.15): now also TP38.1
- net at U4.19 (P0.16): now also TP39.1
- net at U4.2 (P0.00/XL1): now also TP23.1
- net at U4.20 (P0.17): now also TP40.1
- net at U4.21 (P0.18/SWO): now also TP41.1
- net at U4.22 (P0.19): now also TP42.1
- net at U4.23 (P0.20): now also TP43.1
- net at U4.24 (P0.21/~{RESET}): now also TP20.1
- net at U4.27 (P0.22): now also TP44.1
- net at U4.28 (P0.23): now also TP45.1
- net at U4.29 (P0.24): now also TP46.1
- net at U4.3 (P0.01/XL2): now also TP24.1
- net RF: now reaches L3.1, U4.30 (ANT)
- net RF: now also C28.1
- net at U4.37 (P0.25): now also TP47.1
- net at U4.38 (P0.26): now also TP48.1
- net at U4.39 (P0.27): now also TP49.1
- net at U4.4 (P0.02/AIN0): now also TP25.1
- net at U4.40 (P0.28/AIN4): now also TP50.1
- net at U4.41 (P0.29/AIN5): now also TP51.1
- net at U4.42 (P0.30/AIN6): now also TP52.1
- net at U4.43 (P0.31/AIN7): now also TP53.1
- net at U4.5 (P0.03/AIN1): now also TP26.1
- net RF_MATCH: now reaches L3.2
- net RF_MATCH: now also C27.1, FLT1.1 (IN)
- net at R4.1: now also TP5.1; no longer TP2.1
- net +BATT renamed +PWR
- net +PWR: now also TP1.1; no longer TP15.1
- net CS: no longer names the net of U3.39 (*CS)
- net CS: now also TP17.1; no longer U4.9 (P0.07)
- net DRDY: no longer names the net of U3.47 (*DRDY)
- net DRDY: now also TP14.1; no longer U4.6 (P0.04/AIN2)
- net MISO: no longer names the net of U3.43 (DOUT)
- net MISO: now also TP15.1; no longer U4.7 (P0.05/AIN3)
- net MOSI: no longer names the net of U3.34 (DIN)
- net MOSI: now also TP19.1; no longer U4.11 (NFC1/P0.09)
- net RESET: no longer names the net of U4.10 (P0.08)
- net RESET: now also TP31.1; no longer U3.36 (*RESET)
- net SCLK: no longer names the net of U3.40 (SCLK)
- net SCLK: now also TP16.1; no longer U4.14 (P0.11)
- net SWDCLK: no longer names the net of U4.25 (SWDCLK)
- net SWDCLK: now also TP21.1; no longer U4.8 (P0.06)
- net SWDIO: no longer names the net of U4.26 (SWDIO)
- net SWDIO: now also TP22.1
- new net: C11.1, R7.2, U3.9 (IN4N)
- new net: C7.1, R3.2, U3.1 (IN8N)
- new net: C12.1, R8.2, U3.11 (IN3N)
- new net: C13.1, R9.2, U3.13 (IN2N)
- new net: R10.1, U3.15 (IN1N)
- new net: C8.1, R4.2, U3.3 (IN7N)
- new net: TP18.1, U3.36 (*RESET)
- new net: TP32.1, U4.11 (NFC1/P0.09)
- new net: TP28.1, U4.7 (P0.05/AIN3)
- new net: TP34.1, U4.14 (P0.11)
- new net: TP27.1, U4.6 (P0.04/AIN2)
- new net: TP29.1, U4.8 (P0.06)
- new net: TP30.1, U4.9 (P0.07)
- new net RF_ANT: FLT1.3 (OUT), L4.2 (NC)
- now unconnected: C14.2, U3.6 (IN6P)
- no-connect marks 36 -> 14
Other:
- note added: "(32 Mhz)"
- note added: "-2.5V"
- note added: "2.5V"
- note added: "A PWR"
- note added: "BIAS"
- note added: "D PWR"
- note added: "DEBUG"
- note added: "Electrodes"
- note added: "Fiducial Markers"
- note added: "HSE"
- note added: "Mounting Holes (M2)"
- note added: "RF"
- note added: "SPI"
- moved on the sheet: C1, C11, C12, C13, C14, C15, C16, C17, C18, C19, C2, C20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
