File: hardware/kicad/Circuit layout.kicad_sch (KiCad schematic)
At the start: 129 parts, among them U1 TPS7A2025PDQNR, U2 LM27761, U3 ADS1299IPAGR, U4 nRF52832-QFxx, Y1 32MHz

Commit message: Schematic + BOM finished
Parts:
- added R2: 5K, Resistor_SMD:R_0402_1005Metric_Pad0.72x0.64mm_HandSolder, symbol Device:R
- C1, C2, C34, C35, C36, C37, C38, C4, C6: Distributor Link (none) -> https://www.mouser.co.uk/ProductDetail/KYOCERA-AVX/04024D10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; Manufacturer (none) -> KYOCERA AVX; Manufacturer Part Number (none) -> 04024D105KAT2A
- C10: renamed from C9; Distributor Link (none) -> https://www.mouser.co.uk/ProductDetail/Murata-Electronics/G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; Manufacturer (none) -> Murata Electronics; Manufacturer Part Number (none) -> GRM1555C1H472GE01D
- C11: renamed from C10; Distributor Link (none) -> https://www.mouser.co.uk/ProductDetail/Murata-Electronics/G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; Manufacturer (none) -> Murata Electronics; Manufacturer Part Number (none) -> GRM1555C1H472GE01D
- C12: renamed from C11; Distributor Link (none) -> https://www.mouser.co.uk/ProductDetail/Murata-Electronics/G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; Manufacturer (none) -> Murata Electronics; Manufacturer Part Number (none) -> GRM1555C1H472GE01D
- C13: renamed from C12; Distributor Link (none) -> https://www.mouser.co.uk/ProductDetail/Murata-Electronics/G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; Manufacturer (none) -> Murata Electronics; Manufacturer Part Number (none) -> GRM1555C1H472GE01D
- C14: renamed from C13; Distributor Link (none) -> https://www.mouser.co.uk/ProductDetail/Murata-Electronics/G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; Manufacturer (none) -> Murata Electronics; Manufacturer Part Number (none) -> GRM1555C1H472GE01D
- C15: renamed from C14; Distributor Link (none) -> https://www.mouser.co.uk/ProductDetail/Murata-Electronics/G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; Manufacturer (none) -> Murata Electronics; Manufacturer Part Number (none) -> GRM1555C1H472GE01D
- C16: renamed from C15; Distributor Link (none) -> https://www.mouser.co.uk/ProductDetail/KYOCERA-AVX/04026C10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; Manufacturer (none) -> KYOCERA AVX; Manufacturer Part Number (none) -> 04026C104MAT2A
- C17: renamed from C16; Distributor Link (none) -> https://www.mouser.co.uk/ProductDetail/KEMET/C0402C106M7PAC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; Manufacturer (none) -> KEMET; Manufacturer Part Number (none) -> C0402C106M7PAC7867
- C18: renamed from C17; Distributor Link (none) -> https://www.mouser.co.uk/ProductDetail/KYOCERA-AVX/04024D10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; Manufacturer (none) -> KYOCERA AVX; Manufacturer Part Number (none) -> 04024D105KAT2A
- C19: renamed from C18; Distributor Link (none) -> https://www.mouser.co.uk/ProductDetail/Murata-Electronics/G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; Manufacturer (none) -> Murata Electronics; Manufacturer Part Number (none) -> GRM21BR60G107ME11K
- C20: renamed from C19; Distributor Link (none) -> https://www.mouser.co.uk/ProductDetail/KYOCERA-AVX/04024D10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; Manufacturer (none) -> KYOCERA AVX; Manufacturer Part Number (none) -> 04024D105KAT2A
- C21: renamed from C20; Distributor Link (none) -> https://www.mouser.co.uk/ProductDetail/KYOCERA-AVX/04026C15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; Manufacturer (none) -> KYOCERA AVX; Manufacturer Part Number (none) -> 04026C152KAT2A
- C22: renamed from C21; Distributor Link (none) -> https://www.mouser.co.uk/ProductDetail/KYOCERA-AVX/04026C10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; Manufacturer (none) -> KYOCERA AVX; Manufacturer Part Number (none) -> 04026C104MAT2A
- C23: renamed from C22; Distributor Link (none) -> https://www.mouser.co.uk/ProductDetail/KYOCERA-AVX/04024D10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; Manufacturer (none) -> KYOCERA AVX; Manufacturer Part Number (none) -> 04024D105KAT2A
- C24: renamed from C23; Distributor Link (none) -> https://www.mouser.co.uk/ProductDetail/KYOCERA-AVX/04026C10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; Manufacturer (none) -> KYOCERA AVX; Manufacturer Part Number (none) -> 04026C104MAT2A
- C25: renamed from C24; Distributor Link (none) -> https://www.mouser.co.uk/ProductDetail/KYOCERA-AVX/04026C10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; Manufacturer (none) -> KYOCERA AVX; Manufacturer Part Number (none) -> 04026C101KAT2A
- C26: renamed from C25; Distributor Link (none) -> https://www.mouser.co.uk/ProductDetail/KYOCERA-AVX/04024D10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; Manufacturer (none) -> KYOCERA AVX; Manufacturer Part Number (none) -> 04024D105KAT2A
- C27: renamed from C26; Distributor Link (none) -> https://www.mouser.co.uk/ProductDetail/KYOCERA-AVX/04026C10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; Manufacturer (none) -> KYOCERA AVX; Manufacturer Part Number (none) -> 04026C104MAT2A
- C3, C5: Distributor Link (none) -> https://www.mouser.co.uk/ProductDetail/KYOCERA-AVX/CM05X5R4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; Manufacturer (none) -> KYOCERA AVX; Manufacturer Part Number (none) -> CM05X5R475M16AH
- C30: renamed from C29; Distributor Link (none) -> https://www.mouser.co.uk/ProductDetail/KEMET/C0603C120K9RAC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; Manufacturer (none) -> KEMET; Manufacturer Part Number (none) -> C0603C120K9RAC7411
- C31: renamed from C30; Distributor Link (none) -> https://www.mouser.co.uk/ProductDetail/KEMET/C0603C120K9RAC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; Manufacturer (none) -> KEMET; Manufacturer Part Number (none) -> C0603C120K9RAC7411
- C32: renamed from C31; Distributor Link (none) -> https://www.mouser.co.uk/ProductDetail/KYOCERA-AVX/04024D10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; Manufacturer (none) -> KYOCERA AVX; Manufacturer Part Number (none) -> 04024D105KAT2A
- C33: renamed from C32; Distributor Link (none) -> https://www.mouser.co.uk/ProductDetail/KYOCERA-AVX/04024D10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; Manufacturer (none) -> KYOCERA AVX; Manufacturer Part Number (none) -> 04024D105KAT2A
- C7: renamed from C33; Distributor Link (none) -> https://www.mouser.co.uk/ProductDetail/KYOCERA-AVX/04024D10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; Manufacturer (none) -> KYOCERA AVX; Manufacturer Part Number (none) -> 04024D105KAT2A
- C8: renamed from C7; Distributor Link (none) -> https://www.mouser.co.uk/ProductDetail/Murata-Electronics/G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; Manufacturer (none) -> Murata Electronics; Manufacturer Part Number (none) -> GRM1555C1H472GE01D
- C9: renamed from C8; Distributor Link (none) -> https://www.mouser.co.uk/ProductDetail/Murata-Electronics/G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; Manufacturer (none) -> Murata Electronics; Manufacturer Part Number (none) -> GRM1555C1H472GE01D
- FM1, FM2, FM3, H1, H2, H3, H4, TP1, TP10, TP11, TP12, TP13, TP14, TP15, TP16, TP17, TP18, TP19, TP2, TP20, TP21, TP22, TP23, TP24, TP25, TP26, TP27, TP28, TP29, TP3, TP30, TP31, TP32, TP33, TP34, TP35, TP36, TP37, TP38, TP39, TP4, TP40, TP41, TP42, TP43, TP44, TP45, TP46, TP47, TP48, TP49, TP5, TP50, TP51, TP52, TP53, TP54, TP6, TP7, TP8, TP9: now left out of the parts list
- L1: Distributor Link (none) -> https://www.mouser.co.uk/ProductDetail/Murata-Electronics/L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; Manufacturer (none) -> Murata Electronics; Manufacturer Part Number (none) -> LQW15AN15NG8ZD
- L2: Distributor Link (none) -> https://www.mouser.co.uk/ProductDetail/Delevan/S1008R-103J?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; Manufacturer (none) -> Delevan; Manufacturer Part Number (none) -> S1008R-103J
- L4: Distributor Link (none) -> https://www.mouser.co.uk/ProductDetail/ABRACON/AMCA31-2R450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; Manufacturer (none) -> ABRACON; Manufacturer Part Number (none) -> AMCA31-2R450G-S1F-T3
- R1: value 105K -> 100K; Distributor Link (none) -> https://www.mouser.co.uk/ProductDetail/Bourns/CR0402-JW-104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; Manufacturer (none) -> Bourns; Manufacturer Part Number (none) -> CR0402-JW-104GLF
- R10: renamed from R9; value 4.99K -> 5K; Distributor Link (none) -> https://www.mouser.co.uk/ProductDetail/YAGEO/RC0402FR-075KL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; Manufacturer (none) -> YAGEO; Manufacturer Part Number (none) -> RC0402FR-075KL
- R11: renamed from R10; value 4.99K -> 5K; Distributor Link (none) -> https://www.mouser.co.uk/ProductDetail/YAGEO/RC0402FR-075KL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; Manufacturer (none) -> YAGEO; Manufacturer Part Number (none) -> RC0402FR-075KL
- R12: renamed from R11; value 4.99K -> 5K; Distributor Link (none) -> https://www.mouser.co.uk/ProductDetail/YAGEO/RC0402FR-075KL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; Manufacturer (none) -> YAGEO; Manufacturer Part Number (none) -> RC0402FR-075KL
- R13: renamed from R12; Distributor Link (none) -> https://www.mouser.co.uk/ProductDetail/Vishay/CRCW040250K0F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; Manufacturer (none) -> Vishay; Manufacturer Part Number (none) -> CRCW040250K0FKED
- R14: renamed from R13; Distributor Link (none) -> https://www.mouser.co.uk/ProductDetail/Vishay/CRCW04021M00J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; Manufacturer (none) -> Vishay; Manufacturer Part Number (none) -> CRCW04021M00JNTD
- R15: renamed from R13; value 10K -> 1M; Distributor Link (none) -> https://www.mouser.co.uk/ProductDetail/Vishay/CRCW04021M00J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; Manufacturer (none) -> Vishay; Manufacturer Part Number (none) -> CRCW04021M00JNTD
- R16: renamed from R14; Distributor Link (none) -> https://www.mouser.co.uk/ProductDetail/Wurth-Elektronik/560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; Manufacturer (none) -> Wurth Elektronik; Manufacturer Part Number (none) -> 560112110006
- R17: renamed from R15; Distributor Link (none) -> https://www.mouser.co.uk/ProductDetail/Wurth-Elektronik/560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; Manufacturer (none) -> Wurth Elektronik; Manufacturer Part Number (none) -> 560112110006
- R18: renamed from R16; Distributor Link (none) -> https://www.mouser.co.uk/ProductDetail/Wurth-Elektronik/560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; Manufacturer (none) -> Wurth Elektronik; Manufacturer Part Number (none) -> 560112110006
- R19: renamed from R17; Distributor Link (none) -> https://www.mouser.co.uk/ProductDetail/Wurth-Elektronik/560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; Manufacturer (none) -> Wurth Elektronik; Manufacturer Part Number (none) -> 560112110006
- R20: renamed from R18; Distributor Link (none) -> https://www.mouser.co.uk/ProductDetail/Wurth-Elektronik/560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; Manufacturer (none) -> Wurth Elektronik; Manufacturer Part Number (none) -> 560112110006
- R21: renamed from R19; Distributor Link (none) -> https://www.mouser.co.uk/ProductDetail/Wurth-Elektronik/560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; Manufacturer (none) -> Wurth Elektronik; Manufacturer Part Number (none) -> 560112110006
- R3: renamed from R2; Distributor Link (none) -> https://www.mouser.co.uk/ProductDetail/Bourns/CR0402-JW-104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; Manufacturer (none) -> Bourns; Manufacturer Part Number (none) -> CR0402-JW-104GLF
- R4: renamed from R3; value 4.99K -> 5K; Distributor Link (none) -> https://www.mouser.co.uk/ProductDetail/YAGEO/RC0402FR-075KL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; Manufacturer (none) -> YAGEO; Manufacturer Part Number (none) -> RC0402FR-075KL
- R5: renamed from R4; value 4.99K -> 5K; Distributor Link (none) -> https://www.mouser.co.uk/ProductDetail/YAGEO/RC0402FR-075KL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; Manufacturer (none) -> YAGEO; Manufacturer Part Number (none) -> RC0402FR-075KL
- R6: renamed from R5; value 4.99K -> 5K; Distributor Link (none) -> https://www.mouser.co.uk/ProductDetail/YAGEO/RC0402FR-075KL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; Manufacturer (none) -> YAGEO; Manufacturer Part Number (none) -> RC0402FR-075KL
- R7: renamed from R6; value 4.99K -> 5K; Distributor Link (none) -> https://www.mouser.co.uk/ProductDetail/YAGEO/RC0402FR-075KL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; Manufacturer (none) -> YAGEO; Manufacturer Part Number (none) -> RC0402FR-075KL
- R8: renamed from R7; value 4.99K -> 5K; Distributor Link (none) -> https://www.mouser.co.uk/ProductDetail/YAGEO/RC0402FR-075KL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; Manufacturer (none) -> YAGEO; Manufacturer Part Number (none) -> RC0402FR-075KL
- R9: renamed from R8; value 4.99K -> 5K; Distributor Link (none) -> https://www.mouser.co.uk/ProductDetail/YAGEO/RC0402FR-075KL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; Manufacturer (none) -> YAGEO; Manufacturer Part Number (none) -> RC0402FR-075KL
- U1: Distributor Link (none) -> https://www.mouser.co.uk/ProductDetail/Texas-Instruments/TP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; Manufacturer (none) -> Texas Instruments; Manufacturer Part Number (none) -> TPS7A2025PDQNR
- U2: Distributor Link (none) -> https://www.mouser.co.uk/ProductDetail/Texas-Instruments/LM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; Manufacturer (none) -> Texas Instruments; Manufacturer Part Number (none) -> LM27761DSGR
- U3: Distributor Link (none) -> https://www.mouser.co.uk/ProductDetail/Texas-Instruments/AD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; Manufacturer (none) -> Texas Instruments; Manufacturer Part Number (none) -> ADS1299IPAGR
- U4: Distributor Link (none) -> https://www.mouser.co.uk/ProductDetail/Nordic-Semiconductor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; Manufacturer (none) -> Nordic Semiconductor; Manufacturer Part Number (none) -> nRF52832-QFAA-R
- renumbered C27 to C28, C28 to C29
Connections:
- net at R3.1, U2.5 (VFB): now also R2.1; no longer R1.2
- net BIASOUT renamed EEGBIASOUT
- new net: R1.2, R2.2
Other:
- moved on the sheet: TP3, TP54
