File: hardware/pcb_bridge2/pcb_bridge2.kicad_sch (KiCad schematic)
At the start: 2 parts, among them J1 68710614522, J2 687108149022

Commit message: both bridge finished
main pcb layout nearly there
Connections:
- net AVSS: now also J2.3, J2.6; no longer J2.1, J2.8
- net at J1.1: now also J2.8; no longer J2.7
- net at J1.2: now also J2.7; no longer J2.6
- net at J1.5: now also J2.2; no longer J2.3
- net at J1.6: now also J2.1; no longer J2.2
Changed lines of the file:
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@@
-	)
-	(junction
-		(at 85.09 50.8)
-		(diameter 0)
-		(color 0 0 0 0)
 	)
 	(junction
@@
 		(color 0 0 0 0)
 	)
-	(junction
-		(at 93.98 73.66)
-		(diameter 0)
-		(color 0 0 0 0)
-	)
 	(wire
 		(pts
@@
 	(wire
 		(pts
-			(xy 113.03 63.5) (xy 113.03 72.39)
-		)
-		(stroke
-			(width 0)
-			(type default)
-		)
-	)
-	(wire
-		(pts
-			(xy 107.95 46.99) (xy 85.09 46.99)
+			(xy 116.84 53.34) (xy 107.95 53.34)
 		)
 		(stroke
@@
 	(wire
 		(pts
-			(xy 107.95 55.88) (xy 116.84 55.88)
-		)
-		(stroke
-			(width 0)
-			(type default)
-		)
-	)
-	(wire
-		(pts
 			(xy 124.46 49.53) (xy 161.29 49.53)
 		)
@@
 	(wire
 		(pts
-			(xy 107.95 63.5) (xy 113.03 63.5)
-		)
-		(stroke
-			(width 0)
-			(type default)
-		)
-	)
-	(wire
-		(pts
-			(xy 116.84 55.88) (xy 116.84 63.5)
+			(xy 116.84 53.34) (xy 116.84 63.5)
 		)
 		(stroke
@@
 	(wire
 		(pts
+			(xy 107.95 66.04) (xy 113.03 66.04)
+		)
+		(stroke
+			(width 0)
+			(type default)
+		)
+	)
+	(wire
+		(pts
 			(xy 107.95 60.96) (xy 114.3 60.96)
 		)
@@
 	(wire
 		(pts
-			(xy 85.09 46.99) (xy 85.09 50.8)
+			(xy 111.76 68.58) (xy 111.76 74.93)
 		)
 		(stroke
@@
 	(wire
 		(pts
-			(xy 121.92 53.34) (xy 121.92 66.04)
+			(xy 121.92 50.8) (xy 121.92 66.04)
 		)
 		(stroke
@@
 	(wire
 		(pts
+			(xy 107.95 50.8) (xy 121.92 50.8)
+		)
+		(stroke
+			(width 0)
+			(type default)
+		)
+	)
+	(wire
+		(pts
 			(xy 170.18 43.18) (xy 130.81 43.18)
 		)
@@
 	(wire
 		(pts
-			(xy 111.76 66.04) (xy 111.76 74.93)
-		)
-		(stroke
-			(width 0)
-			(type default)
-		)
-	)
-	(wire
-		(pts
 			(xy 107.95 58.42) (xy 115.57 58.42)
 		)
@@
 	(wire
 		(pts
-			(xy 107.95 66.04) (xy 111.76 66.04)
-		)
-		(stroke
-			(width 0)
-			(type default)
-		)
-	)
-	(wire
-		(pts
 			(xy 129.54 55.88) (xy 130.81 55.88)
 		)
@@
 	(wire
 		(pts
-			(xy 107.95 73.66) (xy 107.95 68.58)
-		)
-		(stroke
-			(width 0)
-			(type default)
-		)
-	)
-	(wire
-		(pts
 			(xy 115.57 60.96) (xy 130.81 60.96)
 		)
@@
 	(wire
 		(pts
-			(xy 93.98 73.66) (xy 107.95 73.66)
-		)
-		(stroke
-			(width 0)
-			(type default)
-		)
-	)
-	(wire
-		(pts
-			(xy 107.95 53.34) (xy 121.92 53.34)
-		)
-		(stroke
-			(width 0)
-			(type default)
-		)
-	)
-	(wire
-		(pts
 			(xy 156.21 53.34) (xy 156.21 55.88)
 		)
@@
 	(wire
 		(pts
+			(xy 113.03 66.04) (xy 113.03 72.39)
+		)
+		(stroke
+			(width 0)
+			(type default)
+		)
+	)
+	(wire
+		(pts
 			(xy 161.29 69.85) (xy 114.3 69.85)
 		)
@@
 	(wire
 		(pts
+			(xy 107.95 68.58) (xy 111.76 68.58)
+		)
+		(stroke
+			(width 0)
+			(type default)
+		)
+	)
+	(wire
+		(pts
 			(xy 129.54 46.99) (xy 129.54 55.88)
-		)
-		(stroke
-			(width 0)
-			(type default)
-		)
-	)
-	(wire
-		(pts
-			(xy 107.95 50.8) (xy 107.95 46.99)
 		)
 		(stroke
@@
 					(unit 1)
 				)
+			)
+		)
+	)
+	(symbol
+		(lib_id "power:GND")
+		(at 107.95 55.88 90)
+		(unit 1)
+		(exclude_from_sim no)
+		(in_bom yes)
+		(on_board yes)
+		(dnp no)
+		(fields_autoplaced yes)
+		(property "Reference" "#PWR04"
+			(at 114.3 55.88 0)
+			(effects
+				(font
+					(size 1.27 1.27)
+				)
+				(hide yes)
+			)
+		)
+		(property "Value" "AVSS"
+			(at 111.76 55.8799 90)
+			(effects
+				(font
+					(size 1.27 1.27)
+				)
+				(justify right)
+				(hide yes)
+			)
+		)
+		(property "Footprint" ""
+			(at 107.95 55.88 0)
+			(effects
+				(font
+					(size 1.27 1.27)
+				)
+				(hide yes)
+			)
+		)
+		(property "Datasheet" ""
+			(at 107.95 55.88 0)
+			(effects
+				(font
+					(size 1.27 1.27)
+				)
+				(hide yes)
+			)
+		)
+		(property "Description" "Power symbol creates a global label with name \"GND\" , ground"
+			(at 107.95 55.88 0)
+			(effects
+				(font
+					(size 1.27 1.27)
+				)
+				(hide yes)
+			)
+		)
+		(pin "1"
+		)
+		(instances
+			(project "pcb_bridge2"
+				(path "/c9ffe863-bcda-4bf3-b9ec-ad736cda5403"
+					(reference "#PWR04")
+					(unit 1)
+				)
+			)
+		)
+	)
+	(symbol
+		(lib_id "power:GND")
+		(at 107.95 63.5 90)
+		(unit 1)
+		(exclude_from_sim no)
+		(in_bom yes)
+		(on_board yes)
+		(dnp no)
+		(fields_autoplaced yes)
+		(property "Reference" "#PWR03"
+			(at 114.3 63.5 0)
+			(effects
+				(font
+					(size 1.27 1.27)
+				)
+				(hide yes)
+			)
+		)
+		(property "Value" "AVSS"
+			(at 111.76 63.4999 90)
+			(effects
+				(font
+					(size 1.27 1.27)
+				)
+				(justify right)
+				(hide yes)
+			)
+		)
+		(property "Footprint" ""
+			(at 107.95 63.5 0)
+			(effects
+				(font
+					(size 1.27 1.27)
+				)
+				(hide yes)
+			)
+		)
+		(property "Datasheet" ""
+			(at 107.95 63.5 0)
+			(effects
+				(font
+					(size 1.27 1.27)
+				)
+				(hide yes)
+			)
+		)
+		(property "Description" "Power symbol creates a global label with name \"GND\" , ground"
+			(at 107.95 63.5 0)
+			(effects
+				(font
+					(size 1.27 1.27)
+				)
+				(hide yes)
+			)
+		)
+		(pin "1"
+		)
+		(instances
+			(project "pcb_bridge2"
+				(path "/c9ffe863-bcda-4bf3-b9ec-ad736cda5403"
+					(reference "#PWR03")
+					(unit 1)
+				)
